File: Hardware/AetherPhylax.kicad_sch (KiCad schematic)
At the start: 39 parts, among them J1 Conn_01x01_Pin, J2 Conn_01x01_Pin, U2 BME280, U3 STM32G071KxU, U4 RFM95W-868S2

Commit message: switch to 4Layer Board, fixed I2C Addr
Parts:
- removed DEBUG1: Conn_02x03_Top_Bottom, Library:TestPoint_2x03_P1.27mm, symbol Connector_Generic:Conn_02x03_Top_Bottom
- added DEBUG1: Conn_02x03_Odd_Even, MyLib:TestPoint_2x03_1.5mm, symbol Connector_Generic:Conn_02x03_Odd_Even
- renumbered ROK3 to ROK1, ROK1 to ROK3, ROUT2 to ROUT1, ROUT1 to ROUT2, ROV2 to ROV1, ROV1 to ROV2
Connections:
- net GND: now also U2.5 (SDO), DEBUG1.5 (Pin_5), DEBUG1.6 (Pin_6)
- net RX: now also DEBUG1.4 (Pin_4)
- net SWCLK: now also DEBUG1.3 (Pin_3)
- net SWDIO: now also DEBUG1.1 (Pin_1)
- net TX: now also DEBUG1.2 (Pin_2)
